File: MOS-modules/MOS-MICROPROCESSOR/MOS.sch (KiCad schematic (older format))
At the start: 12 parts, among them J1 Conn_01x03_Male, J2 Conn_01x34_Male, SW1 SW_Push, U1 6502, X1 CXO_DIP8

Commit message: MOS 6503 Rev B
Connections:
- net CLK_INPUT is gone; now on net CLK: J1.2 (Pin_2), U1.37 (ϕ0)
- net CLK: no longer J1.3 (Pin_3)
- net CLK_INTERNAL: now also J1.3 (Pin_3); no longer J1.1 (Pin_1)
Changed lines of the file:
@@
 	5750 3750 5450 3750
 Text Label 5350 2850 0    50   ~ 0
-CLK_INPUT
+CLK
 Text Label 5450 3750 0    50   ~ 0
 RWB
@@
 Wire Wire Line
 	5350 3050 5750 3050
+Wire Wire Line
+	2550 6350 3150 6350
+Text Label 2950 4350 2    50   ~ 0
+CLK_INTERNAL
 Text Label 2950 4250 2    50   ~ 0
-CLK_INPUT
-Wire Wire Line
-	2550 6350 3150 6350
-Text Label 2950 4150 2    50   ~ 0
-CLK_INTERNAL
-Text Label 2950 4350 2    50   ~ 0
 CLK
 Text Label 5350 2950 0    50   ~ 0
